File: Hardware/irtransceiver.kicad_pcb (KiCad board)
At the start: 2 copper layers, 59.9 x 22.2 mm, 15 parts, among them J1 USB_C_Receptacle_USB2.0_16P, U1 ESP32-S3-WROOM-1, U2 AMS1117-3.3

Commit message: hardware/gen: Designed and drew IR emitter driver
Picked parts for bom and placed on PCB view for layout of emitter; Reciever design next.
Parts:
- added D1: Test LED, LED_SMD:LED_0603_1608Metric, F.Cu at (200.5, 102.6)
- added D2: VSMY14940, ethanimports:LED_MY14940_VIS, F.Cu at (195.8, 98.1)
- added Q1: MMBT2222A, Package_TO_SOT_SMD:SOT-23, F.Cu at (200.9, 99.1)
- added R5: 330Ω, Resistor_SMD:R_0805_2012Metric, F.Cu at (194.7, 101.0)
- added R6: 330Ω, Resistor_SMD:R_0603_1608Metric, F.Cu at (203.2, 93.0)
- added R7: 47Ω, Resistor_SMD:R_2512_6332Metric, F.Cu at (196.8, 94.2)
Connections:
- U1 pad 39: unconnected-(U1-IO1-Pad39) -> Net-(U1-IO1)
