File: Hardware/irtransceiver.kicad_sch (KiCad schematic)
At the start: 17 parts, among them J1 USB_C_Receptacle_USB2.0_16P, U1 ESP32-S3-WROOM-1, U2 AMS1117-3.3

Commit message: hardware/schematic: cleared naming isssues with 3v3 rail test LED
Parts:
- D1: value LED -> Test LED
Changed lines of the file:
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@@
 			)
 		)
-		(property "Value" "LED"
+		(property "Value" "Test LED"
 			(at 241.3 118.4274 90)
 			(effects

Commit message: hardware/gen: Designed and drew IR emitter driver
Picked parts for bom and placed on PCB view for layout of emitter; Reciever design next.
Parts:
- added D2: VSMY14940, ethanimports:LED_MY14940_VIS, symbol VSMY14940:VSMY14940
- added Q1: MMBT2222A, Package_TO_SOT_SMD:SOT-23, symbol Transistor_BJT:MMBT2222A
- added R6: 330Ω, Resistor_SMD:R_0603_1608Metric, symbol Device:R_US
- added R7: 47Ω, Resistor_SMD:R_2512_6332Metric, symbol Device:R_US
Connections:
- net +5V: now also R7.1
- net GND: now also Q1.2 (E)
- net at U1.39 (IO1): now also R6.2
- new net: Q1.1 (B), R6.1
- new net: D2.A, R7.2
- new net: D2.C, Q1.3 (C)
Other:
- note added: "Decoupling"
- note added: "IR Driver"
- title: IR Applications -> IR Transceiver
- moved on the sheet: C3, C4
